File: omega.kicad_pcb (KiCad board)
At the start: 2 copper layers, 31.6 x 31.4 mm, 22 parts, among them J1 Conn_01x04_Female, J2 Power TOP, J3 Power BOTTOM, Q1 MMBF5457, Q2 BS170

Commit message: added runoffgroove.com attribution to back silkscreen
Other:
- board text added: "CC BY-NC-SA 3.0"
- board text added: "by runoffgroove.com"
Changed lines of the file:
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@@
     )
   )
-  (property "DATE" "2020-09-05")
+  (property "DATE" "2020-09-23")
   (property "REVISION" "v1.3-1")
   (property "TITLE" "Omega")
@@
   (gr_line (start 96.678 52.324) (end 116.204919 52.324) (layer "Edge.Cuts") (width 0.1))
   (gr_line (start 90.678 58.293) (end 90.678 83.693) (layer "Edge.Cuts") (width 0.1))
-  (gr_text "${TITLE}" (at 99.568 75.438) (layer "B.SilkS")
-    (effects (font (size 1.5 1.5) (thickness 0.3)) (justify mirror))
+  (gr_text "${TITLE}" (at 108.204 64.897 270) (layer "B.SilkS")
+    (effects (font (size 1.4 1.5) (thickness 0.3)) (justify mirror))
+  )
+  (gr_text "by runoffgroove.com" (at 106.553 64.516 270) (layer "B.SilkS")
+    (effects (font (size 0.8 0.8) (thickness 0.127)) (justify mirror))
+  )
+  (gr_text "CC BY-NC-SA 3.0" (at 104.775 64.389 270) (layer "B.SilkS")
+    (effects (font (size 0.8 0.7) (thickness 0.127)) (justify mirror))
   )
   (gr_text "${REVISION}\n${DATE}" (at 117.221 79.375) (layer "B.SilkS")
     (effects (font (size 1 0.9) (thickness 0.127)) (justify mirror))
   )
-  (gr_text "${URL}" (at 91.694 73.787 270) (layer "B.SilkS")
+  (gr_text "${URL}" (at 91.567 73.787 270) (layer "B.SilkS")
     (effects (font (size 0.8 0.8) (thickness 0.127)) (justify mirror))
   )
