File: omega.kicad_sch (KiCad schematic)
At the start: 22 parts, among them J1 Conn_01x04_Female, J2 Power TOP, J3 Power BOTTOM, Q1 MMBF5457, Q2 BS170

Commit message: tighter visual layout, same functionality
Parts:
- J1: value Conn_01x04_Female -> Stomp
Connections:
- net at Q1.1 (D): now also C6.1, RV2.2, RV2.3; no longer R4.2
- new net: Q1.2 (S), R4.2
Other:
- moved on the sheet: C3, D1, D2, J1, J2, J3, R7
